File: condo_schematics_kicad/condo_schematics_kicad.kicad_sch (KiCad schematic)
At the start: 3 parts

Commit message: Adding kicad schematics and PCB
Parts:
- added J10, J11: Conn_01x01_Male, Connector_PinHeader_2.54mm:PinHeader_1x01_P2.54mm_Vertical, symbol Connector:Conn_01x01_Male
- added J2, J4, J6, J8: (no value), symbol Connector:Screw_Terminal_01x02
- added J3, J5, J7, J9: (no value), symbol Connector:Conn_01x01_Male
- added R10, R12, R13, R6, R7, R9: R, Resistor_THT:R_Axial_DIN0207_L6.3mm_D2.5mm_P7.62mm_Horizontal, symbol Device:R
- added R11, R5, R8: 110, Resistor_THT:R_Axial_DIN0207_L6.3mm_D2.5mm_P7.62mm_Horizontal, symbol Device:R
- added R2, R3, R4: (no value), symbol Device:R
- added U1: (no value), symbol Isolator:EL817
- added U2, U3, U4: EL817, Package_DIP:DIP-4_W7.62mm, symbol Isolator:EL817
- D1: value (none) -> DIODE; footprint (none) -> Diode_THT:D_5W_P12.70mm_Horizontal
- J1: value (none) -> Conn_01x02_Male; footprint (none) -> Connector_PinHeader_2.54mm:PinHeader_1x02_P2.54mm_Vertical
- R1: value (none) -> 570; footprint (none) -> Resistor_THT:R_Axial_DIN0207_L6.3mm_D2.5mm_P2.54mm_Vertical
Connections:
- new net: J2.2 (Pin_2), R2.1
- new net: R2.2, U1.1
- new net: R8.2, U3.1
- new net: J6.1 (Pin_1), U3.2
- new net: R10.1, R9.1, U3.3
- new net: R5.2, U2.1
- new net: J4.1 (Pin_1), U2.2
- new net: R6.1, R7.1, U2.3
- new net: J5.1 (Pin_1), R7.2
- new net: R3.1, R4.1, U1.3
- new net: J9.1 (Pin_1), R13.2
- new net: J3.1 (Pin_1), R4.2
- new net: J7.1 (Pin_1), R10.2
- new net: R12.1, R13.1, U4.3
- new net: J2.1 (Pin_1), U1.2
- new net: J8.1 (Pin_1), U4.2
- new net: J8.2 (Pin_2), R11.1
- new net: J4.2 (Pin_2), R5.1
- new net: R11.2, U4.1
- new net: J6.2 (Pin_2), R8.1
- new net +3V3: J11.1 (Pin_1), U1.4, U2.4, U3.4, U4.4
- new net GND: J10.1 (Pin_1), R12.2, R3.2, R6.2, R9.2

Commit message: Cleaning test schematics and PCBs
Parts:
- removed D1: DIODE, Diode_THT:D_5W_P12.70mm_Horizontal, symbol pspice:DIODE
- removed J1: Conn_01x02_Male, Connector_PinHeader_2.54mm:PinHeader_1x02_P2.54mm_Vertical, symbol Connector:Conn_01x02_Male
- removed R1: 570, Resistor_THT:R_Axial_DIN0207_L6.3mm_D2.5mm_P2.54mm_Vertical, symbol Device:R
- J2, J4, J6, J8: value (none) -> Screw_Terminal_01x02; footprint (none) -> TerminalBlock:TerminalBlock_Altech_AK300-2_P5.00mm
- J3, J5, J7, J9: value (none) -> Conn_01x01_Male; footprint (none) -> Connector_PinHeader_2.54mm:PinHeader_1x01_P2.54mm_Vertical
- R2: value (none) -> 110; footprint (none) -> Resistor_THT:R_Axial_DIN0207_L6.3mm_D2.5mm_P7.62mm_Horizontal
- R3, R4: value (none) -> R; footprint (none) -> Resistor_THT:R_Axial_DIN0207_L6.3mm_D2.5mm_P7.62mm_Horizontal
- U1: value (none) -> EL817; footprint (none) -> Package_DIP:DIP-4_W7.62mm
